File: yusynth-minimoog-vcf/minimoog_panel.kicad_pcb (KiCad board)
At the start: 2 copper layers, 30.5 x 128.3 mm, 14 parts

Commit message: Fixed input 2 text on panel
Parts:
- In 2: renamed from In 1
Changed lines of the file:
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@@
   (module PanelMounting:JackMounting_3.5mm (layer B.Cu)
     (at 139.7 114.3 180)
-    (fp_text reference "In 1" (at 0 -6.35 180) (layer B.SilkS)
+    (fp_text reference "In 2" (at 0 -6.35 180) (layer B.SilkS)
       (effects (font (size 1.5 1.5) (thickness 0.3)) (justify mirror))
     )
